Commit message: feat:能够精准跟随的完美身躯(

File: src/arm_description/urdf/dual_arm_shared_load.xacro (robot description, xacro)
@@ -31,5 +31,5 @@
       <mass value="1.0"/>
       <origin xyz="0 0 0"/>
-      <inertia ixx="0.01" ixy="0" ixz="0" iyy="0.01" iyz="0" izz="0.01"/>
+      <inertia ixx="0.00042" ixy="0" ixz="0" iyy="0.1202" iyz="0" izz="0.1202"/>
     </inertial>
     <visual>
